File: pcb/hackpad.kicad_pcb (KiCad board)
At the start: 2 copper layers, 45.5 x 70 mm, 5 parts, among them SW1 SW_Push, SW2 SW_Push, SW3 SW_Push, U1 MOUDLE-SEEEDUINO-XIAO, U2 ER_OLEDM0.91_1x-I2C

Commit message: Add files via upload
Routing:
- net GND: track 54.1 -> 71.9 mm
Changed lines of the file:
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@@
 			(drillshape 0)
 			(scaleselection 1)
-			(outputdirectory "../../../Downloads/gerbers/")
+			(outputdirectory "../../../Downloads/gerbersv2/")
 		)
 	)
@@
 	)
 	(segment
+		(start 120.96 136.46)
+		(end 122.46 137.96)
+		(width 0.2)
+		(layer "F.Cu")
+		(net "GND")
+	)
+	(segment
 		(start 120.96 88.65)
 		(end 125.11 84.5)
 		(width 0.2)
 		(layer "F.Cu")
+		(net "GND")
+	)
+	(segment
+		(start 122.46 137.96)
+		(end 130.75 137.96)
+		(width 0.2)
+		(layer "F.Cu")
+		(net "GND")
+	)
+	(segment
+		(start 120.96 129.15)
+		(end 120.96 136.46)
+		(width 0.2)
+		(layer "F.Cu")
